File: radio-usb.kicad_sch (KiCad schematic)
At the start: 29 parts

Commit message: eagle library
Parts:
- added C?: 100u, symbol Device:C_Polarized
- added C? (x3): 10u, symbol Device:C_Polarized
- added C? (x2): 100n, symbol Device:C
- added D? (x6): CM1213A-01SO, Package_TO_SOT_SMD:SOT-23, symbol Power_Protection:CM1213A-01SO
- added D?: B0530W-7-F, Diode_SMD:D_SOD-123, symbol Device:D_Schottky
- added J?: Barrel_Jack, symbol Connector:Barrel_Jack
- added L?: 1u, symbol Device:L
- added Q?: BC846C, Package_TO_SOT_SMD:SOT-23, symbol Transistor_BJT:BC846
- added R? (x4): 33, symbol Device:R_Small
- added R? (x3): 10k, symbol Device:R
- added R?: 10k, symbol Device:R_Small
- added R?: R_Small, symbol Device:R_Small
- added TP?: +5VP_OK, symbol Connector:TestPoint
- added U?: AP2171W, Package_TO_SOT_SMD:SOT-23-5, symbol Power_Management:AP2171W
- added U? (x2): AP22814AW5, Package_TO_SOT_SMD:SOT-23-5, symbol Power_Management:AP22814AW5
- added U?: L7805, symbol Regulator_Linear:L7805
Connections:
- net D+: now also D?.1 (CH1)
- net D-: now also D?.1 (CH1)
- net GND: now also J?.4 (GND1), J?.8 (GND2), J?.9 (Shield), C?.2, C?.2, C?.2, C?.2, C?.2, C?.2, D?.3 (VN), D?.3 (VN), D?.3 (VN), D?.3 (VN), D?.3 (VN), D?.3 (VN), J?.2, Q?.2 (E), R?.1, U?.2 (GND), U?.2 (GND), U?.2 (GND), U?.2 (GND)
- net VBUS: now also D?.2 (VP), D?.2 (VP), R?.2, U?.5 (IN)
- net at U?.1 (USBDM_DN1/PRT_DIS_M1): no longer U?.2 (D-)
- net at U?.10 (VDDA33): now also U?.29 (VDDA33), U?.36 (VDDA33), U?.5 (VDDA33), C?.1, C?.1, L?.2
- net at U?.15 (VDD33): now also U?.23 (VDD33)
- net at U?.2 (USBDP_DN1/PRT_DIS_P1): no longer U?.1 (D+)
- net H_DP1+: now reaches U?.6 (USBDM_DN3/PRT_DIS_M3)
- net H_DP1+: now also R?.1
- net H_DP1-: now reaches U?.7 (USBDP_DN3/PRT_DIS_P3)
- net H_DP1-: now also R?.1
- net H_DP2-: now reaches U?.8 (USBDM_DN4/PRT_DIS_M4)
- net H_DP2-: now also R?.1
- net H_DP2+: now reaches U?.9 (USBDP_DN4/PRT_DIS_P4)
- net H_DP2+: now also R?.1
- net +5VP: now reaches J?.1 (VBUS1)
- net +5VP: now also J?.5 (VBUS2), D?.2 (VP), D?.2 (VP), D?.2 (VP), D?.2 (VP), U?.1 (OUT)
- net DP1-: now reaches J?.2 (D1-)
- net DP1-: now also D?.1 (CH1), R?.2
- net DP1+: now reaches J?.3 (D1+)
- net DP1+: now also D?.1 (CH1), R?.2
- net DP2-: now reaches J?.6 (D2-)
- net DP2-: now also D?.1 (CH1), R?.2
- net DP2+: now reaches J?.7 (D2+)
- net DP2+: now also D?.1 (CH1), R?.2
- new net: Q?.1 (B), R?.2
- new net: Q?.3 (C), R?.1, U?.4 (EN)
- new net: C?.1, C?.1, R?.2, U?.3 (OUT), U?.4 (EN), U?.5 (IN)
- new net: D?.2 (A), J?.1
- new net +12V: C?.1, D?.1 (K), R?.1, U?.1 (IN)
- new net +5V: C?.1, L?.1, R?.1, R?.2, U?.1 (OUT), U?.1 (OUT), U?.5 (IN)
- new net +5VP_EN: R?.1, U?.4 (EN)
- new net +5VP_OK: R?.2, TP?.1, U?.3 (~{FLG})
Other:
- moved on the sheet: J?, R?, U?

Commit message: daily
Parts:
- added C? (x2): 10p, symbol Device:C
- added C? (x4): 10u, symbol Device:C_Polarized
- added C? (x3): 1u, symbol Device:C_Polarized
- added C? (x3): 1u, symbol Device:C
- added C? (x7): 100n, symbol Device:C
- added C?: 220u, symbol Device:C_Polarized
- added C?: 220uF, symbol Device:C_Polarized
- added C? (x2): 100n, symbol Device:C_Small
- added C?: 3u3, symbol Device:C_Polarized
- added L? (x2): 1u, symbol Device:L
- added Q? (x2): BC846, Package_TO_SOT_SMD:SOT-23, symbol Transistor_BJT:BC846
- added R? (x4): 10k, symbol Device:R
- added R?: 1k, symbol Device:R
- added R? (x4): 22, symbol Device:R
- added R? (x3): 10k, symbol Device:R_Small
- added R?: 12k, symbol Device:R
- added R? (x2): 330, symbol Device:R
- added R? (x3): 0, symbol Device:R
- added R?: 2k2, symbol Device:R
- added R?: 1k5, symbol Device:R
- added R?: 2R2, symbol Device:R
- added R?: 1M, symbol Device:R
- added SW? (x2): SW_DIP_x04, symbol Switch:SW_DIP_x04
- added U?: LM1117-3.3, symbol Regulator_Linear:LM1117-3.3
- added U? (x4): PC817, Package_DIP:DIP-4_W7.62mm, symbol Isolator:PC817
- added U?: MIC5209-3.6YS, Package_TO_SOT_SMD:SOT-223-3_TabPin2, symbol MIC5209:MIC5209-3.3YS
- added U?: 93CxxC, symbol Memory_EEPROM:93CxxC
- added Y?: Crystal, symbol Device:Crystal
- added Y?: 12M, symbol Device:Crystal
- R? (x2): value R_Small -> 22
Connections:
- net +3V3: now also L?.1, R?.2, R?.2, R?.2, R?.2, U?.6 (ORG), U?.8 (VCC)
- net +5V: now also U?.50 (VREGIN), C?.1, R?.1, U?.1 (VIN), U?.3 (VI)
- net GND: now also U?.1 (GND), U?.10 (AGND), U?.11 (AGNDC), U?.11 (GND), U?.13 (TEST), U?.15 (GND), U?.18 (AGNDP), U?.22 (AGNDX), U?.25 (GND), U?.26 (DGND), U?.35 (GND), U?.4 (DGNDU), U?.47 (GND), U?.5 (GND), U?.51 (GND), C?.2, C?.2, C?.2, C?.2, C?.2, C?.2, C?.2, C?.2, C?.2, C?.2, C?.2, C?.2, C?.2, C?.2, C?.2, C?.2, C?.2, C?.2, C?.2, C?.2, C?.2, C?.2, Q?.2 (E), Q?.2 (E), R?.1, R?.1, R?.2, R?.2, R?.2, U?.1 (GND), U?.2 (GND), U?.5 (GND)
- net H_USBDM_SER: now reaches U?.1 (USBDM_DN1/PRT_DIS_M1)
- net H_USBDM_SER: now also R?.1
- net H_USBDP_SER: now reaches U?.2 (USBDP_DN1/PRT_DIS_P1)
- net H_USBDP_SER: now also R?.1
- net H_USBDM_AUD_: now reaches U?.3 (USBDM_DN2/PRT_DIS_M2)
- net H_USBDM_AUD_: now also R?.1
- net H_USBDP_AUD_: now reaches U?.4 (USBDP_DN2/PRT_DIS_P2)
- net H_USBDP_AUD_: now also R?.1, R?.1
- net AUD_USB_DP: now reaches U?.1 (D+)
- net AUD_USB_DP: now also R?.2
- net at U?.10 (VCCCI): now also C?.1, R?.2
- net AUD_IN_LEFT: now reaches U?.12 (VINL)
- net AUD_IN_RIGHT: now reaches U?.13 (VINR)
- net at U?.14 (VCOM): now also C?.1
- net AUD_OUT_RIGHT: now reaches U?.15 (VOUTR)
- net AUD_OUT_RIGHT: now also C?.1
- net AUD_OUT_LEFT: now reaches U?.16 (VOUTL)
- net AUD_OUT_LEFT: now also C?.1
- net at U?.17 (VCCP1I): now also C?.1
- net at U?.19 (VCCP2I): now also C?.1
- net AUD_USB_DN: now reaches U?.2 (D-)
- net AUD_USB_DN: now also R?.2
- net at U?.20 (XTO): now also C?.1, R?.1, Y?.1
- net at U?.21 (XTI): now also C?.1, R?.2, Y?.2
- net at U?.23 (VCCXI): now also C?.1
- net at U?.24 (DIN): now also R?.2
- net at U?.25 (DOUT): now also R?.1
- net AUD_VDDI: now reaches U?.27 (VDDI)
- net AUD_VDDI: now also U?.8 (SEL0), U?.9 (SEL1), C?.1, R?.2
- net AUD_VBUS: now reaches U?.3 (VBUS)
- net AUD_VBUS: now also C?.1, R?.2
- net +1V8: now reaches U?.12 (VCORE)
- net +1V8: now also U?.37 (VCORE), U?.49 (VREGOUT), U?.64 (VCORE), C?.1, C?.1
- net at U?.14 (~{RESET}): now also R?.1
- net SER_A_RTS_OUT: now reaches U?.18 (ADBUS2)
- net SER_A_RTS_OUT: now also R?.1
- net SER_A_CTS_IN: now reaches U?.19 (ADBUS3)
- net SER_A_CTS_IN: now also R?.1, U?.3
- net at U?.2 (OSCI): now also C?.1, Y?.2
- net SER_VCCIO: now reaches U?.20 (VCCIO)
- net SER_VCCIO: now also U?.31 (VCCIO), U?.42 (VCCIO), U?.56 (VCCIO), C?.1, C?.1, C?.1, C?.1, L?.2, R?.2, R?.2, U?.4, U?.4
- net SER_A_DTR_OUT: now reaches U?.21 (ADBUS4)
- net SER_A_DTR_OUT: now also R?.1
- net SER_A_DSR_IN: now reaches U?.22 (ADBUS5)
- net SER_A_DSR_IN: now also R?.1, U?.3
- net at U?.3 (OSCO): now also C?.1, Y?.1
- net SER_B_TXD_OUT: now reaches U?.38 (BDBUS0)
- net SER_B_RXD_IN: now reaches U?.39 (BDBUS1)
- net SER_VPLL: now reaches U?.4 (VPHY)
- net SER_VPLL: now also U?.9 (VPLL), C?.1, C?.1, C?.1, L?.1, L?.2
- net SER_B_RTS_OUT: now reaches U?.40 (BDBUS2)
- net SER_B_CTS_IN: now reaches U?.41 (BDBUS3)
- net SER_B_DTR_OUT: now reaches U?.43 (BDBUS4)
- net SER_B_DSR_IN: now reaches U?.44 (BDBUS5)
- net SER_B_RXLED: now reaches U?.54 (BCBUS3)
- net SER_B_TXLED: now reaches U?.55 (BCBUS4)
- net at U?.6 (REF): now also R?.2
- net at U?.61 (EEDATA): now also R?.1, U?.3 (DI)
- net at U?.62 (EECLK): now also R?.1, U?.2 (SCLK)
- net at U?.63 (EECS): now also R?.1, U?.1 (CS)
- net at U?.7 (DM): now also R?.2
- net at U?.8 (DP): now also R?.2
- new net: Q?.3 (C), U?.2 (x2)
- new net: R?.1, U?.1 (x2)
- new net: R?.1, R?.2, U?.4 (DO)
- new net: C?.1, R?.1, U?.3 (VOUT)
- new net GNDREF: U?.2, U?.2, U?.3, U?.3
- new net PTT_C_DTR_A: Q?.1 (B), R?.2
- new net PTT_C_RTS_A: Q?.1 (B), R?.2
Other:
- moved on the sheet: J?, R?, TP?, U?

Commit message: schematic ready
Parts:
- removed Q?: BC846, Package_TO_SOT_SMD:SOT-23, symbol Transistor_BJT:BC846
- removed R? (x4): 10k, symbol Device:R
- removed R?: 330, symbol Device:R
- removed U? (x2): PC817, Package_DIP:DIP-4_W7.62mm, symbol Isolator:PC817
- added ?, U?: CRIYCHLEY9000, paratnc_cp:NORMAL, symbol paratnc_cp:CRIYCHLEY9000
- added C?: 10u, Capacitor_SMD:C_1206_3216Metric_Pad1.33x1.80mm_HandSolder, symbol Device:C
- added C? (x2): 4u7, Capacitor_SMD:C_0805_2012Metric_Pad1.18x1.45mm_HandSolder, symbol Device:C
- added C? (x2): 100u, Capacitor_THT:CP_Radial_D10.0mm_P5.00mm, symbol Device:C_Polarized
- added C? (x7): 100n, Capacitor_SMD:C_0805_2012Metric_Pad1.18x1.45mm_HandSolder, symbol Device:C
- added C? (x7): 10u, Capacitor_Tantalum_SMD:CP_EIA-3216-18_Kemet-A_Pad1.58x1.35mm_HandSolder, symbol Device:C_Polarized
- added C?: 100n, Capacitor_SMD:C_0805_2012Metric_Pad1.18x1.45mm_HandSolder, symbol Device:C_Small
- added D? (x6): RB751V40T1G, Diode_SMD:D_SOD-323_HandSoldering, symbol Diode:1N6857
- added D? (x2): LED, Capacitor_SMD:C_0805_2012Metric_Pad1.18x1.45mm_HandSolder, symbol Device:LED
- added D?: 1N4148W, Diode_SMD:D_SOD-123, symbol Diode:1N4148W
- added D?: QLS6B-FKW, LED_SMD:LED_Cree-PLCC6_4.7x1.5mm, symbol LED:QLS6B-FKW
- added F?: Polyfuse 100mA, Resistor_SMD:R_1210_3225Metric_Pad1.30x2.65mm_HandSolder, symbol Device:Polyfuse
- added J?: Mini-DIN-6, AV:Mini-DIN_Female_TM0508A, symbol Connector:Mini-DIN-6
- added J? (x2): Conn_Coaxial, AV:rca_cliff_F68371, symbol Connector:Conn_Coaxial
- added J? (x2): ACJS-MHDRM, AV:Jack_6.35mm_ACJS-MHDRM, symbol Connector:AudioJack3_Ground_Switch
- added J?: DB9_Female, Connector_Dsub:DSUB-9_Female_Horizontal_P2.77x2.84mm_EdgePinOffset4.94mm_Housed_MountingHolesOffset7.48mm, symbol Connector:DB9_Female
- added J?: 15EDGRC-3.5-03P-14, Connector_Phoenix_MC:PhoenixContact_MCV_1,5_3-G-3.5_1x03_P3.50mm_Vertical, symbol Connector:Screw_Terminal_01x03
- added J?: DB9_Male, Connector_Dsub:DSUB-9_Male_Horizontal_P2.77x2.84mm_EdgePinOffset4.94mm_Housed_MountingHolesOffset7.48mm, symbol Connector:DB9_Male
- added L? (x2): 4u7, Inductor_SMD:L_1210_3225Metric_Pad1.42x2.65mm_HandSolder, symbol Device:L_Ferrite
- added L?: 1u, Inductor_SMD:L_1210_3225Metric_Pad1.42x2.65mm_HandSolder, symbol Device:L
- added Q?: BC856, Package_TO_SOT_SMD:SOT-23, symbol Transistor_BJT:BC856
- added Q? (x2): BC846, Package_TO_SOT_SMD:SOT-23, symbol Transistor_BJT:BC846
- added R?: 100k, Resistor_SMD:R_0805_2012Metric_Pad1.20x1.40mm_HandSolder, symbol Device:R
- added R? (x6): 660, Resistor_SMD:R_0805_2012Metric_Pad1.20x1.40mm_HandSolder, symbol Device:R
- added R? (x10): 2k2, Resistor_SMD:R_0805_2012Metric_Pad1.20x1.40mm_HandSolder, symbol Device:R
- added R? (x11): 10k, Resistor_SMD:R_0805_2012Metric_Pad1.20x1.40mm_HandSolder, symbol Device:R
- added R? (x2): 0, Resistor_SMD:R_0805_2012Metric_Pad1.20x1.40mm_HandSolder, symbol Device:R
- added R? (x5): 620, Resistor_SMD:R_0805_2012Metric_Pad1.20x1.40mm_HandSolder, symbol Device:R
- added R?: 22k, Resistor_SMD:R_0805_2012Metric_Pad1.20x1.40mm_HandSolder, symbol Device:R
- added R?: 4k7, Resistor_SMD:R_0805_2012Metric_Pad1.20x1.40mm_HandSolder, symbol Device:R
- added R?: 330, Resistor_SMD:R_0805_2012Metric_Pad1.20x1.40mm_HandSolder, symbol Device:R
- added RN?: 10k, Resistor_THT:R_Array_SIP5, symbol Device:R_Network04
- added RV?: 10k, potentiometers:Potentiometer_SRpassives_1028F, symbol Device:R_Potentiometer
- added SW? (x2): SW_DPDT_x2, switches_spdt_dpdt:Alps_SSSS222700, symbol Switch:SW_DPDT_x2
- added SW? (x2): SW_SPDT, switches_spdt_dpdt:Alps_SSSS213000, symbol Switch:SW_SPDT
- added SW?: SW_SPDT, switches_spdt_dpdt:TL3XWO, symbol Switch:SW_SPDT
- added SW?: SW_Push_DPDT, switches_spdt_dpdt:Alps_SSSS222700, symbol Switch:SW_Push_DPDT
- added TP?: TTL_RX, TestPoint:TestPoint_Pad_D2.0mm, symbol Connector:TestPoint
- added TP?: TTL_TX_2, TestPoint:TestPoint_Pad_D2.0mm, symbol Connector:TestPoint
- added TP?: +12V_FLG, TestPoint:TestPoint_Pad_D2.0mm, symbol Connector:TestPoint
- added TP?: TTL_TX, TestPoint:TestPoint_Pad_D2.0mm, symbol Connector:TestPoint
- added TP?: SER_B_TXD_OUT, TestPoint:TestPoint_Pad_D2.0mm, symbol Connector:TestPoint
- added TP?: TTL_RX_2, TestPoint:TestPoint_Pad_D2.0mm, symbol Connector:TestPoint
- added TP?: VB_FLG, TestPoint:TestPoint_Pad_D2.0mm, symbol Connector:TestPoint
- added TP?: SER_B_RXD_IN, TestPoint:TestPoint_Pad_D2.0mm, symbol Connector:TestPoint
- added U? (x7): 4069, Package_SO:SOIC-14_3.9x8.7mm_P1.27mm, symbol 4xxx:4069
- added U?: PC817, Package_DIP:DIP-4_W7.62mm, symbol Isolator:PC817
- added U? (x2): LMV358, Package_SO:SOIC-8_3.9x4.9mm_P1.27mm, symbol Amplifier_Operational:LMV358
- added U?: TBA 1-0511, Converter_DCDC:Converter_DCDC_Murata_CRE1xxxxxx3C_THT, symbol Regulator_Switching:CRE1S0305S3C
- added U? (x2): TLP2662, Package_SO:SOIC-8_3.9x4.9mm_P1.27mm, symbol Isolator:HCPL-0630
- added U?: MAX3232, Package_SO:SOIC-16_3.9x9.9mm_P1.27mm, symbol Interface_UART:MAX3232
- added U?: 24LC04, Package_DIP:DIP-8_W7.62mm, symbol Memory_EEPROM:24LC04
- added X?: MAB5SH, sterownik:MAB5SH, symbol sterownik-eagle:MAB5SH
- C? (x25): footprint (none) -> Capacitor_SMD:C_0805_2012Metric_Pad1.18x1.45mm_HandSolder
- C? (x7): footprint (none) -> Capacitor_Tantalum_SMD:CP_EIA-3216-18_Kemet-A_Pad1.58x1.35mm_HandSolder; DESCRIPTION (none) -> TPSA106K010R0900 KYOCERA AVX
- C?: footprint (none) -> Capacitor_THT:CP_Radial_D10.0mm_P5.00mm; DESCRIPTION (none) -> UBT1H101MPD8 NICHICON
- C?: value 220u -> 10u; footprint (none) -> Capacitor_Tantalum_SMD:CP_EIA-3216-18_Kemet-A_Pad1.58x1.35mm_HandSolder; DESCRIPTION (none) -> TPSA106K010R0900 KYOCERA AVX
- C?: value 220uF -> 10u; footprint (none) -> Capacitor_Tantalum_SMD:CP_EIA-3216-18_Kemet-A_Pad1.58x1.35mm_HandSolder; DESCRIPTION (none) -> TPSA106K010R0900 KYOCERA AVX
- D? (x2): value LED -> LED_HS; footprint (none) -> Capacitor_SMD:C_0805_2012Metric_Pad1.18x1.45mm_HandSolder
- D?: value LED -> LED_ACTIVE; footprint (none) -> Capacitor_SMD:C_0805_2012Metric_Pad1.18x1.45mm_HandSolder
- J?: footprint (none) -> Connector_BarrelJack:BarrelJack_GCT_DCJ200-10-A_Horizontal
- L? (x3): footprint (none) -> Inductor_SMD:L_1210_3225Metric_Pad1.42x2.65mm_HandSolder
- R? (x41): footprint (none) -> Resistor_SMD:R_0805_2012Metric_Pad1.20x1.40mm_HandSolder
- SW? (x2): footprint (none) -> Button_Switch_SMD:SW_DIP_SPSTx04_Slide_Copal_CHS-04B_W7.62mm_P1.27mm
- TP?: footprint (none) -> TestPoint:TestPoint_Pad_D2.0mm
- U?: footprint (none) -> Package_TO_SOT_SMD:TO-252-2
- U?: footprint (none) -> Package_TO_SOT_THT:TO-220-3_Horizontal_TabDown
- U?: footprint (none) -> Package_DIP:DIP-8_W7.62mm
- Y? (x3): footprint (none) -> Crystal:Crystal_SMD_HC49-SD_HandSoldering
Connections:
- net +3V3: now also L?.1, U?.2 (VO), C?.1, U?.8 (VCC)
- net +5V: now also C?.1, D?.1 (AB), D?.3 (AR), D?.5 (AG), L?.1, L?.1; no longer L?.1, R?.1
- net AUD_IN_LEFT: now also C?.1
- net AUD_IN_RIGHT: now also C?.1
- net AUD_VBUS: now also C?.1, C?.1, R?.2, U?.8 (V+)
- net GND: now also ?.P$4, C?.2, C?.2, C?.2, C?.2, C?.2, J?.2 (Ext), J?.2 (Ext), J?.S, J?.S, J?.SN, J?.SN, Q?.2 (E), Q?.2 (E), R?.1, R?.1, R?.1, R?.1, R?.2, RN?.1 (common), RV?.3, U?.1 (-VIN), U?.1 (A0), U?.2 (A1), U?.3 (A2), U?.4 (GND), U?.4 (V-), U?.5 (GND), U?.7 (WP), U?.P$2
- net GNDREF: now also U?.2, ?.P$2, C?.1, C?.2, C?.2, C?.2, C?.2, C?.2, J?.2, J?.3 (Pin_3), J?.5, J?.7, R?.2, U?.15 (GND), U?.3 (-VOUT), U?.5, U?.5 (GND), U?.7 (VSS), U?.9, U?.P$4, X?.2, X?.PE, X?.PE@ (PE); no longer U?.3
- net H_REM1: now also R?.2
- net H_SEL0: now also R?.2
- net SER_A_CTS_IN: now also SW?.1, RN?.5 (R4)
- net SER_A_DSR_IN: now also SW?.2, RN?.4 (R3)
- net SER_A_DTR_OUT: now also SW?.2
- net SER_A_RTS_OUT: now also SW?.1
- net SER_B_CTS_IN: now also SW?.3, RN?.3 (R2)
- net SER_B_DSR_IN: now also SW?.4, RN?.2 (R1)
- net SER_B_DTR_OUT: now also SW?.4
- net SER_B_RTS_OUT: now also SW?.3
- net SER_B_RXD_IN: now also D?.1 (K), D?.1 (K), R?.2, TP?.1
- net SER_B_RXLED: now also D?.2 (A)
- net SER_B_TXD_OUT: now also TP?.1, U?.2 (C1), U?.3 (C2)
- net SER_B_TXLED: now also D?.2 (A)
- net SER_VCCIO: now also U?.4, R?.1, R?.1, R?.2, R?.2, R?.2, SW?.3 (C), U?.8 (VCC)
- net at C?.1, C?.1, L?.2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: now also U?.15 (VDD33), U?.23 (VDD33)
- net RX_ACT_SEP: now reaches SW?.5
- net RX_ACT_SEP: now also SW?.6, SW?.7, SW?.8, U?.3, R?.2
- net at U?.1: now also SW?.2 (B)
- net at U?.3 (~{FLG}): now also TP?.1 (x2)
- net RCA_LEFT: now reaches C?.2
- net RCA_LEFT: now also C?.2, J?.1 (In)
- net RCA_RIGHT: now reaches C?.2
- net RCA_RIGHT: now also C?.2, J?.1 (In)
- net at Q?.3 (C), U?.2: now also U?.2
- net PTT_ACTL: now reaches U?.4
- net PTT_ACTL: now also SW?.1 (A)
- net at SW?.5: now also D?.2 (A)
- net at SW?.6: now also D?.2 (A)
- net at SW?.7: now also D?.2 (A)
- net at SW?.8: now also D?.2 (A)
- net PTT_C_RTS_A: no longer names the net of Q?.1 (B)
- net PTT_C_RTS_A: now also R?.2
- new net: Q?.2 (E), R?.1
- new net: Q?.1 (B), R?.1 (x2)
- new net: R?.2, U?.12
- new net: D?.1 (K), R?.2 (x6)
- new net: U?.2, U?.3
- new net: C?.1, R?.2, U?.1
- new net: C?.2, J?.T
- new net: C?.2, R?.1
- new net: C?.2, R?.2
- new net: C?.1, F?.1, L?.2
- new net: Q?.3 (C), SW?.1 (A)
- new net: R?.2, SW?.3 (C)
- new net: C?.1, J?.R
- new net: ?.P$3, C?.2
- new net: R?.2, U?.1 (A1)
- new net: Q?.1 (B), R?.1, SW?.4 (A)
- new net: R?.1, SW?.6 (C)
- new net: U?.10, U?.13
- new net: R?.1, U?.1
- new net: C?.1, C?.2, L?.1, U?.4 (+VOUT)
- new net: C?.1, U?.6 (VS-)
- new net: C?.1, U?.4 (C2+)
- new net: C?.2, U?.5 (C2-)
- new net: C?.1, L?.2, U?.2 (+VIN)
- new net: J?.R, R?.1, R?.2
- new net: D?.2 (A), R?.1, U?.6 (VO2)
- new net: D?.2 (A), R?.1, U?.7 (VO1)
- new net: R?.1, U?.3 (+)
- new net: R?.1, R?.2, R?.2
- new net: R?.1, U?.5 (SDA)
- new net: D?.4 (KR), R?.1
- new net: L?.2, R?.1
- new net: C?.1, R?.1 (x2)
- new net: R?.1, R?.2, R?.2, U?.2 (-)
- new net: R?.1, U?.2 (C1)
- new net: R?.1, U?.3 (C2)
- new net: Q?.3 (C), R?.2 (x2)
- new net: D?.1 (K), R?.1, SW?.2 (B)
- new net: C?.2, U?.P$3
- new net: C?.1, U?.1 (C1+)
- new net: C?.2, U?.3 (C1-)
- new net: D?.2 (KB), R?.1
- new net: C?.1, U?.2 (VS+)
- new net: J?.RN, J?.TN (x2)
- new net: J?.T, RV?.2
- new net: R?.1, U?.6 (SCL)
- new net: RV?.1, U?.P$1
- new net: D?.6 (KR), R?.1
- new net: R?.2, U?.4 (A2)
- new net AUD_FRM_RADIO: C?.1, J?.3, SW?.2 (B), X?.4
- new net AUD_TO_RADIO: ?.P$1, J?.1, J?.5, X?.1
- new net CAT_UART_RX: J?.1 (Pin_1), SW?.6 (C), U?.1
- new net CAT_UART_TX: J?.2 (Pin_2), R?.1, SW?.3 (C)
- new net PTT: D?.2 (A), J?.3, J?.4, R?.2, SW?.2 (B), SW?.5 (B), X?.3
- new net PTT_ACTH: R?.1, SW?.3 (C), U?.3
- new net PTT_CTRL: R?.1, R?.1, R?.1, R?.1, R?.1, R?.2, SW?.2 (B)
- new net RS232RX: J?.2, U?.13 (R1IN)
- new net RS232TX: J?.3, U?.14 (T1OUT)
- new net RX_ACTIVE: J?.1, J?.6, SW?.5 (B), X?.5
- new net TTL_RX: R?.2, TP?.1, U?.12 (R1OUT)
- new net TTL_RX_2: R?.2, TP?.1, U?.4
- new net TTL_TX: R?.1, TP?.1, U?.11 (T1IN), U?.6 (VO2)
- new net TTL_TX_2: R?.1, TP?.1, U?.11, U?.7 (VO1)
- new net VD: C?.1, F?.2, R?.2, R?.2, R?.2, R?.2, U?.1 (A1), U?.14 (VDD), U?.16 (VCC), U?.4, U?.4 (A2), U?.8 (VCC)
- new net YAESU_FILTERED_AUD: J?.5, SW?.1 (A)
- new net YAESU_FLAT_AUD: J?.4, SW?.3 (C)
Other:
- note added: "INSERT"
- note added: "ISOLATED"
- moved on the sheet: C?, Q?, R?, SW?, U?

Commit message: routing usb differential pairs
Parts:
- added H1, H2, H3, H4: MountingHole, MountingHole:MountingHole_3.2mm_M3, symbol Mechanical:MountingHole
- D13: renamed from D?; footprint LED_SMD:LED_Cree-PLCC6_4.7x1.5mm -> LED:LED_MENTOR_1882
- J1: renamed from J?; value USB_B -> miniUSB
- J10, J11: renamed from J?; symbol Connector:AudioJack3_Ground_Switch -> Connector:AudioJack3_Switch
- J3: renamed from J?; footprint Connector_Phoenix_MC:PhoenixContact_MCV_1,5_3-G-3.5_1x03_P3.50mm_Vertical -> Connector_Phoenix_MC:PhoenixContact_MC_1,5_3-G-3.5_1x03_P3.50mm_Horizontal
- R12, R13, R23, R25, R30, R31: renamed from R?; footprint Resistor_SMD:R_0805_2012Metric_Pad1.20x1.40mm_HandSolder -> Resistor_SMD:R_0603_1608Metric_Pad0.98x0.95mm_HandSolder
- X1: renamed from X?; footprint sterownik:MAB5SH -> sterownik-eagle:MAB5SH
- gave numbers to parts that had none: 209
Connections:
- net AUD_OUT_SUM: now reaches C52.2, J11.T
- net H_VDD: now reaches C10.1, C11.1, L1.2, U5.10 (VDDA33), U5.15 (VDD33), U5.23 (VDD33), U5.29 (VDDA33), U5.36 (VDDA33), U5.5 (VDDA33)
- net AUD_IN_SUM: now reaches J10.R, R61.1, R62.2
- net H_USBDM_AUD_ renamed H_AUD_USBD-
- net H_USBDM_HOST renamed H_HOST_USBD-
- net H_USBDM_SER renamed H_SER_USBD-
- net H_USBDP_AUD_ renamed H_AUD_USBD+
- net H_USBDP_HOST renamed H_HOST_USBD+
- net H_USBDP_SER renamed H_SER_USBD+

Commit message: routing serial ftdi controller
Parts:
- removed R17, R19, R57: 0, Resistor_SMD:R_0805_2012Metric_Pad1.20x1.40mm_HandSolder, symbol Device:R
- removed R5: 10k, Resistor_SMD:R_0805_2012Metric_Pad1.20x1.40mm_HandSolder, symbol Device:R
- added C10: 10u, Capacitor_Tantalum_SMD:CP_EIA-3216-18_Kemet-A_Pad1.58x1.35mm_HandSolder, symbol Device:C_Polarized
- added C13, C23, C24: 100n, Capacitor_SMD:C_0805_2012Metric_Pad1.18x1.45mm_HandSolder, symbol Device:C
- added C38: 470u, Capacitor_THT:CP_Radial_D8.0mm_P3.50mm, symbol Device:C_Polarized
- added J5: EEP_EN, Connector_PinHeader_2.54mm:PinHeader_2x02_P2.54mm_Vertical, symbol Connector_Generic:Conn_02x02_Odd_Even
- added R18, R20: 10k, Resistor_SMD:R_0805_2012Metric_Pad1.20x1.40mm_HandSolder, symbol Device:R
- added U3: APX809_810-xxSA, Package_TO_SOT_SMD:SOT-23_Handsoldering, symbol vdd_supervisor:APX809_810-xxSA
- C28: renamed from C24; value 100n -> 27pF
- C29: renamed from C25; value 100n -> 27pF
- C37: renamed from C33; value 1u -> 100n
- L5: value 1u -> 4u7; DESCRIPTION (none) -> Viking NLV10MTC4R7
- R43: renamed from R44; footprint Resistor_SMD:R_0805_2012Metric_Pad1.20x1.40mm_HandSolder -> Resistor_SMD:R_0603_1608Metric_Pad0.98x0.95mm_HandSolder
- R45: renamed from R46; footprint Resistor_SMD:R_0805_2012Metric_Pad1.20x1.40mm_HandSolder -> Resistor_SMD:R_0603_1608Metric_Pad0.98x0.95mm_HandSolder
- R46: renamed from R47; footprint Resistor_SMD:R_0805_2012Metric_Pad1.20x1.40mm_HandSolder -> Resistor_SMD:R_0603_1608Metric_Pad0.98x0.95mm_HandSolder
- R47: renamed from R50; footprint Resistor_SMD:R_0805_2012Metric_Pad1.20x1.40mm_HandSolder -> Resistor_SMD:R_0603_1608Metric_Pad0.98x0.95mm_HandSolder
- R6: renamed from R7; value 10k -> 100k
- Y1: value Crystal_Small -> 24MHz; footprint Crystal:Crystal_SMD_HC49-SD_HandSoldering -> Crystal:Crystal_SMD_Abracon_ABM8G-4Pin_3.2x2.5mm; DESCRIPTION (none) -> IQD LFXTAL032817BULK
- Y2: value Crystal -> 12MHz; footprint Crystal:Crystal_SMD_HC49-SD_HandSoldering -> Crystal:Crystal_SMD_Abracon_ABM8G-4Pin_3.2x2.5mm
- renumbered C10 to C11, C11 to C12, C12 to C14, C13 to C15, C14 to C16, C15 to C17, C16 to C18, C17 to C19, C18 to C20, C19 to C21, C20 to C22, C21 to C25, C22 to C26, C23 to C27, C26 to C30, C27 to C31, C28 to C32, C29 to C33, C30 to C34, C31 to C35, C32 to C36, C34 to C39, C35 to C40, C36 to C41, C37 to C42, C38 to C43, C39 to C44, C40 to C45, C41 to C46, C42 to C47, C43 to C48, C44 to C49, C45 to C50, C46 to C51, C47 to C52, C48 to C53, C49 to C54, C50 to C55, C51 to C56, C52 to C57, C53 to C58, C54 to C59, C7 to C6, C55 to C60, C6 to C7, D9 to D10, D13 to D12, D12 to D13, D10 to D8, D8 to D9, J9 to J10, J10 to J11, J11 to J12, J5 to J6, J6 to J7, J7 to J8, J8 to J9, R11 to R10, R12 to R11, R13 to R12, R14 to R13, R15 to R14, R16 to R15, R18 to R16, R20 to R17, R21 to R19, R22 to R21, R23 to R22, R24 to R23, R25 to R24, R26 to R25, R30 to R26, R31 to R30, R35 to R31, R38 to R35, R39 to R36, R40 to R37, R36 to R38, R37 to R39, R41 to R40, R42 to R41, R43 to R42, R45 to R44, R6 to R5, R51 to R50, R52 to R51, R53 to R52, R54 to R53, R55 to R54, R56 to R55, R58 to R56, R59 to R57, R60 to R58, R61 to R59, R62 to R60, R63 to R61, R64 to R62, R65 to R63, R66 to R64, R67 to R65, R68 to R66, R69 to R67, R70 to R68, R71 to R69, R8 to R7, R72 to R70, R73 to R71, R74 to R72, R75 to R73, R76 to R74, R77 to R75, R78 to R76, R79 to R77, R9 to R8, R10 to R9, U11 to U10, U9 to U11, U10 to U12, U12 to U13, U13 to U14, U14 to U15, U15 to U16, U16 to U17, U17 to U18, U18 to U19, U19 to U20, U20 to U21, U21 to U22, U22 to U23, U3 to U4, U4 to U5, U5 to U6, U6 to U7, U7 to U8, U8 to U9
Connections:
- net +1V8: now also C23.1, C24.1
- net +3V3: now also R18.2, R20.2; no longer R15.1, R6.1
- net +5V: no longer U17.50 (VREGIN)
- net AUD_VBUS: now also C38.1
- net GND: now also R6.1, C10.2, C13.2, C23.2, C24.2, C38.2, U3.1 (GND); no longer D8.3 (VN)
- net H_AUD_USBD+: now also U6.9 (USBDP_DN4/PRT_DIS_P4); no longer U6.4 (USBDP_DN2/PRT_DIS_P2)
- net H_AUD_USBD-: now also U6.8 (USBDM_DN4/PRT_DIS_M4); no longer U6.3 (USBDM_DN2/PRT_DIS_M2)
- net H_DP1+: now also R30.1, U6.2 (USBDP_DN1/PRT_DIS_P1); no longer R26.1, U6.6 (USBDM_DN3/PRT_DIS_M3)
- net H_DP1-: now also R26.1, U6.1 (USBDM_DN1/PRT_DIS_M1); no longer R30.1, U6.7 (USBDP_DN3/PRT_DIS_P3)
- net H_DP2+: now also U6.4 (USBDP_DN2/PRT_DIS_P2); no longer U6.9 (USBDP_DN4/PRT_DIS_P4)
- net H_DP2-: now also U6.3 (USBDM_DN2/PRT_DIS_M2); no longer U6.8 (USBDM_DN4/PRT_DIS_M4)
- net H_REM1: now also J5.2 (Pin_2)
- net H_RST: now also U3.2 (~{RST})
- net H_SEL0: now also J5.4 (Pin_4)
- net H_SER_USBD+: now also U6.7 (USBDP_DN3/PRT_DIS_P3); no longer U6.2 (USBDP_DN1/PRT_DIS_P1)
- net H_SER_USBD-: now also U6.6 (USBDM_DN3/PRT_DIS_M3); no longer U6.1 (USBDM_DN1/PRT_DIS_M1)
- net H_VDD: now also R15.1, C10.1, C13.1, U3.3 (Vcc)
- net SER_VCCIO: now also U17.50 (VREGIN)
- net ~{SER_RST}: now reaches R51.1, U17.14 (~{RESET})
- net SER_XO: now reaches C29.1, U17.3 (OSCO), Y2.1
- net SER_XI: now reaches C28.1, U17.2 (OSCI), Y2.2
- net SER_EECS: now reaches R52.1, U14.1 (CS), U17.63 (EECS)
- net SER_EEDT: now reaches R49.1, U14.3 (DI), U17.61 (EEDATA)
- net SER_D-: now reaches R47.2, U17.7 (DM)
- net SER_D+: now reaches R45.2, U17.8 (DP)
- net H_EE_SDA: now reaches U2.5 (SDA)
- net H_EE_SDA: now also J5.1 (Pin_1), R18.1
- net H_EE_SCL: now reaches U2.6 (SCL)
- net H_EE_SCL: now also J5.3 (Pin_3), R20.1
Other:
- moved on the sheet: C6, D11, D12, D13, D14, D8, J7, Q2, Q3, R22, R23, R24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
