File: radio-usb.kicad_pcb (KiCad board)
At the start: 2 copper layers, 127 x 90 mm, 225 parts, among them J1 miniUSB, J10 ACJS-MHDRM, J11 ACJS-MHDRM, J2 Barrel_Jack, J3 15EDGRC-3.5-03P-14, J4 DB9_Female, J5 Mini-DIN-6, J6 EDAC 690-008-221-904, J7 DB9_Male, J8 Conn_Coaxial, J9 Conn_Coaxial, Q1 BC846C, Q2 BC846, Q3 BC846, Q4 BC846, Q5 BC856, SW1 SW_Push_DPDT, SW2 SW_SPDT, SW3 SW_SPDT, SW4 SW_DIP_x04, SW5 SW_DIP_x04, SW6 SW_DPDT_x2, SW7 SW_SPDT, U1 L7805, U10 TLP2662, U11 AP2171W, U12 MAX3232, U13 93CxxC, U14 PCM2902, U15 MIC5209-3.6YS, U16 FT2232HL, U17 PC817, U18 CRIYCHLEY9000, U19 PC817, U2 24LC04, U20 PC817, U21 CRIYCHLEY9000, U22 LMV358, U3 AP22814AW5, U4 AP22814AW5, U5 USB2514B_Bi, U6 LM1117-3.3, U7 TBA 1-0511, U8 4069, U9 TLP2662, X1 MAB5SH, Y1 Crystal_Small, Y2 Crystal, Y3 12M

Commit message: routing serial ftdi controller
Parts:
- removed the R17 at (488.2, 116.3)
- removed the R19 at (483.6, 120.8)
- removed the R5 at (499.8, 107.0)
- removed the R57 at (434.6, 171.6)
- added C10: 10u, Capacitor_Tantalum_SMD:CP_EIA-3216-18_Kemet-A_Pad1.58x1.35mm_HandSolder, F.Cu at (70.9, 50.2)
- added C13: 100n, Capacitor_SMD:C_0805_2012Metric_Pad1.18x1.45mm_HandSolder, F.Cu at (68.0, 57.6)
- added C23: 100n, Capacitor_SMD:C_0805_2012Metric_Pad1.18x1.45mm_HandSolder, F.Cu at (101.4, 86.0)
- added C24: 100n, Capacitor_SMD:C_0805_2012Metric_Pad1.18x1.45mm_HandSolder, F.Cu at (86.3, 85.8)
- added C38: 470u, Capacitor_THT:CP_Radial_D8.0mm_P3.50mm, F.Cu at (413.6, 134.3)
- added J5: EEP_EN, Connector_PinHeader_2.54mm:PinHeader_2x02_P2.54mm_Vertical, F.Cu at (85.2, 50.9)
- added R18: 10k, Resistor_SMD:R_0805_2012Metric_Pad1.20x1.40mm_HandSolder, F.Cu at (87.8, 44.5)
- added R20: 10k, Resistor_SMD:R_0805_2012Metric_Pad1.20x1.40mm_HandSolder, F.Cu at (92.4, 44.2)
- added U3: APX809_810-xxSA, Package_TO_SOT_SMD:SOT-23_Handsoldering, F.Cu at (51.1, 46.6)
- C28: renamed from C24; value 100n -> 27pF
- C29: renamed from C25; value 100n -> 27pF
- C37: renamed from C33; value 1u -> 100n
- L5: value 1u -> 4u7
- R43: renamed from R44; footprint Resistor_SMD:R_0805_2012Metric_Pad1.20x1.40mm_HandSolder -> Resistor_SMD:R_0603_1608Metric_Pad0.98x0.95mm_HandSolder
- R45: renamed from R46; footprint Resistor_SMD:R_0805_2012Metric_Pad1.20x1.40mm_HandSolder -> Resistor_SMD:R_0603_1608Metric_Pad0.98x0.95mm_HandSolder
- R46: renamed from R47; footprint Resistor_SMD:R_0805_2012Metric_Pad1.20x1.40mm_HandSolder -> Resistor_SMD:R_0603_1608Metric_Pad0.98x0.95mm_HandSolder
- R47: renamed from R50; footprint Resistor_SMD:R_0805_2012Metric_Pad1.20x1.40mm_HandSolder -> Resistor_SMD:R_0603_1608Metric_Pad0.98x0.95mm_HandSolder
- R6: renamed from R7; value 10k -> 100k
- Y1: value Crystal_Small -> 24MHz; footprint Crystal:Crystal_SMD_HC49-SD_HandSoldering -> Crystal:Crystal_SMD_Abracon_ABM8G-4Pin_3.2x2.5mm
- Y2: value Crystal -> 12MHz; footprint Crystal:Crystal_SMD_HC49-SD_HandSoldering -> Crystal:Crystal_SMD_Abracon_ABM8G-4Pin_3.2x2.5mm
- moved R5 452.3 mm to (51.2, 54.2)
- moved R1 448.4 mm to (45.7, 48.5)
- moved C4 440.2 mm to (45.8, 54.9), turned to 180 degrees
- moved D1 437.2 mm to (42.1, 52.7)
- moved R47 426.5 mm to (63.0, 65.1), turned to -45 degrees
- moved R14 426.2 mm to (50.2, 51.2), turned to 90 degrees
- moved R13 417.6 mm to (52.1, 51.2), turned to -90 degrees
- moved C6 415.6 mm to (56.5, 47.4), turned to -90 degrees
- moved R7 410.4 mm to (66.4, 48.0), turned to 180 degrees
- moved R15 406.8 mm to (54.5, 47.3), turned to -90 degrees
- moved C11 404.7 mm to (66.5, 52.3)
- moved C8 403.9 mm to (70.9, 55.2), turned to -90 degrees
- moved C1 402.0 mm to (45.8, 61.2), turned to 180 degrees
- moved R2 400.0 mm to (74.7, 49.5), turned to 90 degrees
- moved R8 398.8 mm to (66.4, 44.9), turned to 180 degrees
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- renumbered C10 to C11, C11 to C12, C12 to C14, C13 to C15, C14 to C16, C15 to C17, C16 to C18, C17 to C19, C18 to C20, C19 to C21, C20 to C22, C21 to C25, C22 to C26, C23 to C27, C26 to C30, C27 to C31, C28 to C32, C29 to C33, C30 to C34, C31 to C35, C32 to C36, C34 to C39, C35 to C40, C36 to C41, C37 to C42, C38 to C43, C39 to C44, C40 to C45, C41 to C46, C42 to C47, C43 to C48, C44 to C49, C45 to C50, C46 to C51, C47 to C52, C48 to C53, C49 to C54, C50 to C55, C51 to C56, C52 to C57, C53 to C58, C54 to C59, C7 to C6, C55 to C60, C6 to C7, D9 to D10, D13 to D12, D12 to D13, D10 to D8, D8 to D9, J9 to J10, J10 to J11, J11 to J12, J5 to J6, J6 to J7, J7 to J8, J8 to J9, R11 to R10, R12 to R11, R13 to R12, R14 to R13, R15 to R14, R16 to R15, R18 to R16, R20 to R17, R21 to R19, R22 to R21, R23 to R22, R24 to R23, R25 to R24, R26 to R25, R30 to R26, R31 to R30, R35 to R31, R38 to R35, R39 to R36, R40 to R37, R36 to R38, R37 to R39, R41 to R40, R42 to R41, R43 to R42, R45 to R44, R6 to R5, R51 to R50, R52 to R51, R53 to R52, R54 to R53, R55 to R54, R56 to R55, R58 to R56, R59 to R57, R60 to R58, R61 to R59, R62 to R60, R63 to R61, R64 to R62, R65 to R63, R66 to R64, R67 to R65, R68 to R66, R69 to R67, R70 to R68, R71 to R69, R8 to R7, R72 to R70, R73 to R71, R74 to R72, R75 to R73, R76 to R74, R77 to R75, R78 to R76, R79 to R77, R9 to R8, R10 to R9, U11 to U10, U9 to U11, U10 to U12, U12 to U13, U13 to U14, U14 to U15, U15 to U16, U16 to U17, U17 to U18, U18 to U19, U19 to U20, U20 to U21, U21 to U22, U22 to U23, U3 to U4, U4 to U5, U5 to U6, U6 to U7, U7 to U8, U8 to U9
Connections:
- net Net-(C24-Pad1) renamed /SER_XI
- net Net-(C25-Pad1) renamed /SER_XO
- net Net-(R46-Pad2) renamed /SER_D+
- net Net-(R49-Pad1) renamed /SER_EEDT
- net Net-(R50-Pad2) renamed /SER_D-
- net Net-(R52-Pad1) renamed /~{SER_RST}
- net Net-(R53-Pad1) renamed /SER_EECS
- D8 pad 3: GND -> unconnected-(D8-Pad3)
- R15 pad 1: +3V3 -> /H_VDD
- R26 pad 1: /H_DP1+ -> /H_DP1-
- R30 pad 1: /H_DP1- -> /H_DP1+
- R6 pad 1: +3V3 -> GND
- U15 pad 25: Net-(R57-Pad1) -> unconnected-(U15-Pad25)
- U17 pad 50: +5V -> /SER_VCCIO
- U2 pad 5: Net-(R17-Pad1) -> /H_EE_SDA
- U2 pad 6: Net-(R19-Pad1) -> /H_EE_SCL
- U6 pad 1: /H_SER_USBD- -> /H_DP1-
- U6 pad 2: /H_SER_USBD+ -> /H_DP1+
- U6 pad 3: /H_AUD_USBD- -> /H_DP2-
- U6 pad 4: /H_AUD_USBD+ -> /H_DP2+
- U6 pad 6: /H_DP1+ -> /H_SER_USBD-
- U6 pad 7: /H_DP1- -> /H_SER_USBD+
- U6 pad 8: /H_DP2- -> /H_AUD_USBD-
- U6 pad 9: /H_DP2+ -> /H_AUD_USBD+
Routing:
- net /SER_VCCIO: track 0.00 -> 96.0 mm, vias 0 -> 4
- net /H_VDD: track 2.65 -> 96.4 mm, vias 0 -> 10
- net +1V8: track 0.00 -> 89.3 mm, vias 0 -> 3
- net +3V3: track 0.00 -> 50.7 mm, vias 0 -> 4
- net /SER_D-: track 0.00 -> 43.2 mm, vias 0 -> 2
- net /SER_D+: track 0.00 -> 42.0 mm, vias 0 -> 2
- net /SER_VPLL: track 0.00 -> 35.1 mm, vias 0 -> 2
- net /SER_B_CTS_IN: track 0.00 -> 33.8 mm, vias 0 -> 1
- net /SER_B_DTR_OUT: track 0.00 -> 33.3 mm, vias 0 -> 1
- net /SER_B_DSR_IN: track 0.00 -> 31.7 mm, vias 0 -> 1
- net /H_SEL1: track 0.00 -> 30.6 mm, vias 0 -> 2
- net /SER_B_TXLED: track 0.00 -> 30.4 mm, vias 0 -> 2
- net GND: track 0.00 -> 28.7 mm, vias 0 -> 61
- net /SER_B_RXLED: track 0.00 -> 27.8 mm, vias 0 -> 2
- net /H_SEL0: track 0.00 -> 27.1 mm, vias 0 -> 2
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Other:
- board text added: "ACTIVE"
- board text added: "EEPROM ENABLE"
- board text added: "HIGH SPD"
- board text added: "SERIAL RX"
- board text added: "SERIAL TX"

Commit message: daily
Parts:
- D1, D15, D16, D4, D5: footprint Capacitor_SMD:C_0805_2012Metric_Pad1.18x1.45mm_HandSolder -> LED_SMD:LED_0805_2012Metric_Pad1.15x1.40mm_HandSolder
- D6: value B0530W-7-F -> B130-13-F; footprint Diode_SMD:D_SOD-123 -> Diode_SMD:D_SMA
- U1: footprint Package_TO_SOT_THT:TO-220-3_Horizontal_TabDown -> Package_TO_SOT_THT:TO-220-3_Vertical
- U11, U12: footprint Package_SO:SOIC-8_3.9x4.9mm_P1.27mm -> Package_DIP:DIP-8_W7.62mm
- Y3: footprint Crystal:Crystal_SMD_HC49-SD_HandSoldering -> Crystal:Crystal_SMD_Abracon_ABM8G-4Pin_3.2x2.5mm
- moved C7 418.8 mm to (44.5, 39.5), turned to -90 degrees
- moved U5 414.7 mm to (29.8, 57.3), turned to 180 degrees
- moved U4 412.5 mm to (27.0, 53.8), turned to 180 degrees
- moved D6 409.5 mm to (64.9, 30.1), turned to -90 degrees
- moved C9 395.4 mm to (45.5, 43.1), turned to 180 degrees
- moved Q1 395.0 mm to (25.7, 57.3), turned to 180 degrees
- moved C2 385.1 mm to (40.6, 32.9), turned to 90 degrees
- moved R48 369.5 mm to (126.5, 100.5), turned to 90 degrees
- moved R50 355.2 mm to (124.9, 97.6)
- moved C35 339.3 mm to (123.4, 50.5)
- moved U1 335.3 mm to (41.7, 43.5), turned to 90 degrees
- moved R52 334.4 mm to (123.4, 94.3)
- moved C37 329.3 mm to (125.0, 47.1), turned to -90 degrees
- moved R49 298.7 mm to (123.5, 100.9)
- moved C38 296.0 mm to (130.5, 47.9), turned to -90 degrees
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Routing:
- net /SER_EEDT: track 0.00 -> 69.1 mm, vias 0 -> 2
- net Net-(R50-Pad1): track 0.00 -> 68.5 mm, vias 0 -> 2
- net /SER_A_DSR_IN: track 0.00 -> 65.6 mm, vias 0 -> 2
- net /SER_EECS: track 0.00 -> 64.3 mm, vias 0 -> 2
- net /SER_A_CTS_IN: track 1.51 -> 63.4 mm, vias 0 -> 3
- net /SER_B_RTS_OUT: track 4.81 -> 64.0 mm, vias 0 -> 2
- net /SER_B_TXD_OUT: track 5.81 -> 56.3 mm, vias 0 -> 1
- net /SER_B_RXD_IN: track 4.12 -> 53.6 mm, vias 0 -> 1
- net /AUD_USB_DN: track 8.75 -> 47.1 mm
- net /SER_B_CTS_IN: track 33.8 -> 71.4 mm, vias 1 -> 2
- net /SER_A_DTR_OUT: track 1.54 -> 38.8 mm, vias 0 -> 2
- net /AUD_USB_DP: track 8.17 -> 45.4 mm
- net /SER_B_DTR_OUT: track 33.3 -> 63.6 mm, vias 1 -> 2
- net /SER_A_RTS_OUT: track 0.00 -> 29.8 mm, vias 0 -> 2
- net /SER_B_DSR_IN: track 31.7 -> 58.3 mm, vias 1 -> 2
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Other:
- board text added: "A CTS"
- board text added: "A DSR"
- board text added: "A DTR"
- board text added: "A RTS"
- board text added: "B CTS"
- board text added: "B DSR"
- board text added: "B DTR"
- board text added: "B RTS"
- board text added: "PTT"
- board text added: "RX ACT"

Commit message: everything but audio codec
Parts:
- removed the R19 at (418.4, 182.7)
- added C1: 100n, Capacitor_SMD:C_0805_2012Metric_Pad1.18x1.45mm_HandSolder, F.Cu at (48.4, 66.5)
- added C19: 100u, Capacitor_Tantalum_SMD:CP_EIA-3528-21_Kemet-B_Pad1.50x2.35mm_HandSolder, F.Cu at (400.3, 157.8)
- added C54: 22n, Capacitor_SMD:C_0805_2012Metric_Pad1.18x1.45mm_HandSolder, F.Cu at (193.2, 91.3)
- added C56: 22n, Capacitor_SMD:C_0805_2012Metric_Pad1.18x1.45mm_HandSolder, F.Cu at (193.2, 94.3)
- added R20: 0R68, Resistor_SMD:R_1206_3216Metric_Pad1.30x1.75mm_HandSolder, F.Cu at (406.4, 157.3)
- added R58: 16R, Resistor_SMD:R_0805_2012Metric_Pad1.20x1.40mm_HandSolder, F.Cu at (198.0, 94.2)
- added R60: 16R, Resistor_SMD:R_0805_2012Metric_Pad1.20x1.40mm_HandSolder, F.Cu at (198.0, 91.3)
- C15: renamed from C14; footprint Capacitor_THT:CP_Radial_D10.0mm_P5.00mm -> Capacitor_THT:CP_Radial_D5.0mm_P2.50mm
- C16: renamed from C15; value 10u -> 22u
- C18: renamed from C17; value 10u -> 22u
- C20: renamed from C18; value 10u -> 22u
- C23: renamed from C21; value 10u -> 22u
- C24: renamed from C22; footprint Capacitor_SMD:C_0805_2012Metric_Pad1.18x1.45mm_HandSolder -> Capacitor_SMD:C_0603_1608Metric_Pad1.08x0.95mm_HandSolder
- C29: renamed from C27; footprint Capacitor_SMD:C_0805_2012Metric_Pad1.18x1.45mm_HandSolder -> Capacitor_SMD:C_0603_1608Metric_Pad1.08x0.95mm_HandSolder
- C3: renamed from C2; footprint Capacitor_Tantalum_SMD:CP_EIA-3216-18_Kemet-A_Pad1.58x1.35mm_HandSolder -> Capacitor_Tantalum_SMD:CP_EIA-6032-28_Kemet-C_Pad2.25x2.35mm_HandSolder
- C32: renamed from C30; footprint Capacitor_SMD:C_0805_2012Metric_Pad1.18x1.45mm_HandSolder -> Capacitor_SMD:C_0603_1608Metric_Pad1.08x0.95mm_HandSolder
- C33: renamed from C31; footprint Capacitor_SMD:C_0805_2012Metric_Pad1.18x1.45mm_HandSolder -> Capacitor_SMD:C_0603_1608Metric_Pad1.08x0.95mm_HandSolder
- C62: renamed from C58; value 100u -> 220u; footprint Capacitor_THT:CP_Radial_D10.0mm_P5.00mm -> Capacitor_THT:CP_Radial_D6.3mm_P2.50mm
- C63: renamed from C59; value 100u -> 220u; footprint Capacitor_THT:CP_Radial_D10.0mm_P5.00mm -> Capacitor_THT:CP_Radial_D6.3mm_P2.50mm
- R17: footprint Resistor_SMD:R_0805_2012Metric_Pad1.20x1.40mm_HandSolder -> Resistor_SMD:R_0603_1608Metric_Pad0.98x0.95mm_HandSolder
- U1: footprint Package_TO_SOT_THT:TO-220-3_Vertical -> Package_TO_SOT_THT:TO-220-3_Horizontal_TabDown
- U13: footprint Package_SO:SOIC-16_3.9x9.9mm_P1.27mm -> Package_SO:TSSOP-16_4.4x5mm_P0.65mm
- U23: footprint Package_SO:SOIC-8_3.9x4.9mm_P1.27mm -> Package_SO:TSSOP-8_4.4x3mm_P0.65mm
- U9: footprint Package_SO:SOIC-14_3.9x8.7mm_P1.27mm -> Package_SO:TSSOP-14_4.4x5mm_P0.65mm
- moved TP1 441.6 mm to (40.2, 33.7)
- moved R16 426.1 mm to (44.1, 44.1), turned to 90 degrees
- moved C17 410.9 mm to (31.4, 35.4)
- moved TP2 403.1 mm to (43.0, 40.9)
- moved R17 401.2 mm to (46.6, 37.7)
- moved Q5 356.6 mm to (124.7, 86.4)
- moved C15 352.7 mm to (103.4, 47.6), turned to 180 degrees
- moved R78 346.5 mm to (121.1, 88.9), turned to -90 degrees
- moved R28 346.2 mm to (133.9, 87.4), turned to 90 degrees
- moved SW6 336.0 mm to (128.6, 92.7), turned to -90 degrees
- moved R25 328.9 mm to (133.8, 95.2), turned to -90 degrees
- moved R39 325.7 mm to (150.2, 89.9), turned to 180 degrees
- moved R79 325.4 mm to (118.1, 85.8)
- moved R27 320.9 mm to (134.0, 79.6), turned to 90 degrees
- moved R21 313.9 mm to (129.6, 99.7)
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- renumbered C9 to C10, C10 to C11, C11 to C12, C12 to C13, C13 to C14, C16 to C17, C1 to C2, C20 to C21, C19 to C22, C23 to C25, C24 to C26, C25 to C27, C26 to C28, C28 to C30, C29 to C31, C32 to C34, C33 to C35, C34 to C36, C35 to C37, C36 to C38, C37 to C39, C3 to C4, C38 to C40, C39 to C41, C40 to C42, C41 to C43, C42 to C44, C43 to C45, C44 to C46, C45 to C47, C46 to C48, C47 to C49, C4 to C5, C48 to C50, C49 to C51, C50 to C52, C51 to C53, C52 to C55, C53 to C57, C54 to C58, C55 to C59, C5 to C6, C56 to C60, C57 to C61, C60 to C64, C6 to C7, C7 to C8, C8 to C9, D6 to D4, D4 to D5, D5 to D6, J2 to J1, J1 to J2, R20 to R19, R44 to R42, R42 to R43, R43 to R44, R51 to R47, R47 to R48, R48 to R49, R49 to R50, R50 to R51, R58 to R59, R59 to R61, R60 to R62, R61 to R63, R62 to R64, R63 to R65, R64 to R66, R65 to R67, R66 to R68, R67 to R69, R68 to R70, R69 to R71, R70 to R72, R71 to R73, R72 to R74, R73 to R75, R74 to R76, R75 to R77, R76 to R78, R77 to R79
Connections:
- net Net-(C7-Pad1) renamed /5VD12
Routing:
- net +5V: track 0.00 -> 100.5 mm, vias 0 -> 2
- net +12V: track 0.00 -> 85.1 mm, vias 0 -> 2
- net GND: track 50.3 -> 112.5 mm, vias 62 -> 64
- net +3V3: track 57.3 -> 108.5 mm, vias 4 -> 6
- net /5VD12: track 0.00 -> 36.9 mm
- net Net-(D4-Pad2): track 0.00 -> 26.0 mm
- net Net-(R49-Pad1): track 22.8 -> 0.00 mm, vias 1 -> 0
- net VBUS: track 0.00 -> 21.5 mm, vias 0 -> 2
- net /SER_EEDT: track 69.1 -> 84.5 mm
- net /SER_D+: track 42.0 -> 27.5 mm
- net /SER_D-: track 43.2 -> 28.7 mm
- net /SER_EECS: track 64.3 -> 76.5 mm
- net Net-(Q1-Pad3): track 0.00 -> 9.97 mm, vias 0 -> 2
- net /SER_B_TXLED: track 49.6 -> 40.1 mm, vias 4 -> 2
- net Net-(R51-Pad1): track 68.5 -> 77.7 mm
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Other:
- board text added: "OD"
- board text added: "PP"
- board text added: "RX"
- board text added: "SERIAL"
- board text added: "TX"
- board text added: "YAESU UART"
- board text removed: "SERIAL RX"
- board text removed: "SERIAL TX"

Commit message: some components around audio codec
Parts:
- U18, U20, U21: footprint Package_DIP:DIP-4_W7.62mm -> Package_DIP:SMDIP-4_W7.62mm
- moved R54 373.5 mm to (122.8, 53.1), turned to 180 degrees
- moved R43 351.7 mm to (110.3, 47.5), turned to 90 degrees
- moved L5 349.0 mm to (110.4, 39.9), turned to -90 degrees
- moved R53 333.5 mm to (111.9, 43.7)
- moved U21 332.9 mm to (129.3, 72.7), turned to 90 degrees
- moved C27 326.1 mm to (126.9, 52.5)
- moved C61 314.9 mm to (123.9, 66.2), turned to 180 degrees
- moved C49 310.2 mm to (123.3, 63.8)
- moved C53 306.4 mm to (123.3, 61.5)
- moved C50 57.1 mm to (130.0, 56.4)
- moved C51 57.1 mm to (130.0, 58.5)
- moved R55 57.1 mm to (125.9, 57.5)
- moved Y3 57.1 mm to (123.2, 57.4)
- moved SW2 8.48 mm to (128.1, 44.9), turned to 90 degrees
- moved U18 4.14 mm to (121.2, 81.1)
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Connections:
- R43 pad 1: /H_AUD_USBD+ -> /AUD_USB_DP
- R44 pad 1: /H_AUD_USBD- -> /H_AUD_USBD+
- R44 pad 2: /AUD_USB_DN -> /AUD_USB_DP
- R46 pad 1: /H_AUD_USBD+ -> /H_AUD_USBD-
- R46 pad 2: /AUD_USB_DP -> /AUD_USB_DN
Routing:
- net GND: track 112.5 -> 177.4 mm
- net /RCA_LEFT: track 0.00 -> 56.8 mm
- net /RCA_RIGHT: track 0.00 -> 49.6 mm
- net Net-(J11-PadT): track 0.00 -> 32.2 mm, vias 0 -> 1
- net /AUD_IN_SUM: track 0.00 -> 30.2 mm, vias 0 -> 1
- net /AUD_OUT_SUM: track 0.00 -> 23.5 mm
- net Net-(C62-Pad1): track 0.00 -> 21.6 mm
- net /AUD_USB_DP: track 40.3 -> 48.5 mm
- net /AUD_USB_DN: track 40.3 -> 48.4 mm
- net Net-(J12-PadRN): track 0.00 -> 6.20 mm
- net Net-(J11-PadRN): track 0.00 -> 6.20 mm
- net /SER_D+: track 27.5 -> 28.6 mm
Other:
- board text added: "ACT H"
- board text added: "ACT L"

Commit message: daily
Parts:
- removed the C43 at (395.0, 196.8)
- removed F1: Polyfuse 100mA, Resistor_SMD:R_1210_3225Metric_Pad1.30x2.65mm_HandSolder
- removed R56: 0, Resistor_SMD:R_0805_2012Metric_Pad1.20x1.40mm_HandSolder
- removed the R71 at (474.1, 126.9)
- removed the R72 at (474.0, 129.9)
- removed R73, R74: 2k2, Resistor_SMD:R_0805_2012Metric_Pad1.20x1.40mm_HandSolder
- removed RV1: 10k, potentiometers:Potentiometer_SRpassives_1028F
- removed U16: MIC5209-3.6YS, Package_TO_SOT_SMD:SOT-223-3_TabPin2
- added R69: 0, Resistor_SMD:R_0603_1608Metric_Pad0.98x0.95mm_HandSolder, F.Cu at (134.4, 44.5)
- added R70: DNP, Resistor_SMD:R_0603_1608Metric_Pad0.98x0.95mm_HandSolder, F.Cu at (134.5, 51.1)
- R78: renamed from R76; footprint Resistor_SMD:R_0805_2012Metric_Pad1.20x1.40mm_HandSolder -> Resistor_SMD:R_0603_1608Metric_Pad0.98x0.95mm_HandSolder
- U23: value LMV358 -> LMV321IDBVR; footprint Package_SO:TSSOP-8_4.4x3mm_P0.65mm -> Package_TO_SOT_SMD:SOT-23-5_HandSoldering
- moved D13 454.6 mm to (18.0, 88.3)
- moved R23 421.8 mm to (19.5, 73.6)
- moved D8 416.5 mm to (17.5, 104.5)
- moved R34 408.7 mm to (18.9, 80.7)
- moved D2 406.5 mm to (56.9, 21.0)
- moved D3 405.3 mm to (63.7, 20.4)
- moved U10 402.1 mm to (26.0, 80.9)
- moved D11 400.3 mm to (22.6, 96.8)
- moved D14 391.5 mm to (24.1, 90.7)
- moved R61 369.7 mm to (105.0, 59.6), turned to 90 degrees
- moved R57 366.4 mm to (92.4, 63.0)
- moved R59 359.5 mm to (92.4, 64.9)
- moved R64 356.4 mm to (111.3, 47.1)
- moved R63 353.1 mm to (134.0, 74.0), turned to 90 degrees
- moved R9 349.0 mm to (148.2, 90.6), turned to -90 degrees
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- renumbered C42 to C43, C44 to C45, C45 to C46, C46 to C47, C47 to C48, C48 to C49, C49 to C50, C50 to C51, C51 to C52, C52 to C53, C53 to C54, C54 to C55, C55 to C56, C56 to C57, C57 to C58, C58 to C59, C59 to C60, C60 to C61, C61 to C62, C62 to C63, C63 to C64, C64 to C65, R44 to R42, R46 to R43, R42 to R44, R43 to R45, R45 to R46, R69 to R71, R70 to R72, R75 to R77, R77 to R79, R78 to R80, R79 to R81
Connections:
- C23 pad 1: Net-(C23-Pad1) -> VD
- C62 pad 1: Net-(C61-Pad1) (its old number) -> Net-(C62-Pad1)
- D17 pad 1: Net-(D17-Pad1) -> /PTT_CTRL
- D18 pad 1: Net-(D18-Pad1) -> /PTT_CTRL
- D19 pad 1: Net-(D19-Pad1) -> /PTT_CTRL
- D20 pad 1: Net-(D20-Pad1) -> /PTT_CTRL
- L3 pad 2: Net-(C23-Pad1) -> VD
- R71 pad 1: Net-(R69-Pad1) -> Net-(R71-Pad1)
- R77 pad 2: Net-(C61-Pad1) (its old number) -> Net-(C62-Pad1)
- U23 pad 1: Net-(C61-Pad1) (its old number) -> Net-(R71-Pad1)
- U23 pad 2: Net-(R67-Pad2) -> GND
- U23 pad 3: Net-(R69-Pad1) -> Net-(R67-Pad2)
- U23 pad 4: GND -> Net-(C62-Pad1)
- U23 pad 5: (no net) -> /AUD_VBUS
Routing:
- net /AUD_OUT_SUM: track 23.5 -> 84.7 mm
- net Net-(C63-Pad1): track 21.6 -> 70.9 mm
- net /AUD_IN_SUM: track 30.2 -> 70.5 mm
- net Net-(J11-PadT): track 32.2 -> 71.9 mm
- net /RCA_RIGHT: track 49.6 -> 43.1 mm
- net +3V3: track 108.5 -> 102.7 mm
- net /RCA_LEFT: track 56.8 -> 51.6 mm
- net /SER_VPLL: track 35.3 -> 40.4 mm
- net GND: track 177.4 -> 179.3 mm, vias 64 -> 67
- net Net-(C52-Pad1): track 4.99 -> 3.89 mm
- net Net-(C51-Pad1): track 4.98 -> 3.89 mm

Commit message: all components placed
Parts:
- removed C65: 100n, Capacitor_SMD:C_0805_2012Metric_Pad1.18x1.45mm_HandSolder
- D11, D8, TP2, TP4, TP5, TP7, TP8, TP9: moved to B.Cu
- R35, R36, R37: footprint Resistor_SMD:R_0805_2012Metric_Pad1.20x1.40mm_HandSolder -> Resistor_SMD:R_0603_1608Metric_Pad0.98x0.95mm_HandSolder
- moved R68 383.7 mm to (111.3, 64.2), turned to 90 degrees
- moved TP3 355.9 mm to (41.4, 97.0)
- moved TP4 353.3 mm to (140.9, 83.3), turned to 180 degrees
- moved TP8 349.1 mm to (141.8, 75.0), turned to 180 degrees
- moved R77 348.2 mm to (114.9, 66.7)
- moved C33 322.7 mm to (163.2, 91.3)
- moved TP9 320.8 mm to (139.6, 92.7), turned to 180 degrees
- moved C32 318.6 mm to (159.7, 89.6), turned to 180 degrees
- moved C61 315.5 mm to (123.4, 68.9)
- moved C22 314.9 mm to (162.8, 106.1), turned to 180 degrees
- moved TP5 289.6 mm to (148.2, 91.4), turned to 180 degrees
- moved TP7 251.5 mm to (147.1, 97.1), turned to 180 degrees
- moved C60 54.3 mm to (121.7, 72.4), turned to 90 degrees
- moved D11 41.0 mm to (63.6, 95.1), turned to 180 degrees
- moved R23 39.4 mm to (46.4, 102.4), turned to 90 degrees
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Connections:
- net Net-(C18-Pad1) renamed /DCDC_IN
- net Net-(C20-Pad1) renamed /DCDC_OUT
Routing:
- net +3V3: track 102.7 -> 133.1 mm, vias 6 -> 8
- net +5V: track 100.5 -> 87.9 mm
- net /SER_B_TXD_OUT: track 56.3 -> 46.4 mm
- net /SER_B_RXD_IN: track 53.6 -> 47.9 mm
- net GND: track 179.3 -> 174.4 mm
- net /AUD_VBUS: track 12.7 -> 8.70 mm
- net /SER_B_RTS_OUT: track 62.8 -> 60.5 mm
- net /SER_A_CTS_IN: track 63.4 -> 64.7 mm
