File: radio-usb.kicad_pcb (KiCad board)
At the start: 2 copper layers, 127 x 90 mm, 233 parts, among them J1 Barrel_Jack, J10 Conn_Coaxial, J11 ACJS-MHDRM, J12 ACJS-MHDRM, J2 miniUSB, J3 15EDGRC-3.5-03P-14, J4 DB9_Female, J5 EEP_EN, J6 Mini-DIN-6, J7 EDAC 690-008-221-904, J8 DB9_Male, J9 Conn_Coaxial, Q1 BC846C, Q2 BC846C, Q3 BC846C, Q4 BC846C, Q5 BC856, SW1 SW_Push_DPDT, SW2 SW_SPDT, SW3 SW_SPDT, SW4 SW_DIP_x04, SW5 SW_DIP_x04, SW6 SW_DPDT_x2, SW7 SW_SPDT, U1 L7805, U10 AP2171W, U11 TLP2662, U12 TLP2662, U13 MAX3232, U14 93CxxC, U15 PCM2900CDB, U17 FT2232HL, U18 PC817, U19 CRIYCHLEY9000, U2 24LC04, U20 PC817, U21 PC817, U22 CRIYCHLEY9000, U23 LMV321IDBVR, U3 APX809_810-xxSA, U4 AP22814AW5, U5 AP22814AW5, U6 USB2514B-AEZC, U7 LM1117-3.3, U8 TBA 1-0511, U9 4069, X1 MAB5SH, Y1 24MHz, Y2 12MHz, Y3 12M

Commit message: gerber exports and another files sent to PCBway for production
Parts:
- C30, C31: value 30pF -> 18p
- C51, C52: value 10p -> 18p
- D12: value QLS6B-FKW -> 1882.2781
- Y3: value 12M -> 12MHz
- moved Y1 0.36 mm to (45.7, 58.1)
Connections:
- Y1 pad 2: /H_XTALO -> unconnected-(Y1-Pad2)
- Y1 pad 3: (no net) -> /H_XTALO
- Y1 pad 4: (no net) -> GND
- Y2 pad 1: /SER_XO -> GND
- Y2 pad 3: (no net) -> unconnected-(Y2-Pad3)
- Y2 pad 4: (no net) -> /SER_XO
- Y3 pad 2: Net-(C51-Pad1) -> unconnected-(Y3-Pad2)
- Y3 pad 3: (no net) -> Net-(C51-Pad1)
- Y3 pad 4: (no net) -> GND
Routing:
- net GND: track 1110.2 -> 1120.1 mm
- net /H_XTALO: track 12.8 -> 15.4 mm, vias 0 -> 2
- net /SER_XO: track 11.5 -> 10.2 mm, vias 0 -> 2
- net Net-(C51-Pad1): track 11.3 -> 10.5 mm

Commit message: hardware revision b schematic
Parts:
- moved J11 0.45 mm to (88.5, 96.5)
Routing:
- net /AF_FRM_RADIO_PREINS: track 125.9 -> 90.4 mm
- net /AUD_IN_SUM: track 119.8 -> 95.1 mm
- net GND: track 1120.1 -> 1095.6 mm, vias 128 -> 127
- net /RCA_LEFT: track 88.2 -> 98.9 mm, vias 3 -> 4
- net /RCA_RIGHT: track 76.3 -> 85.5 mm, vias 1 -> 2
- net /SER_EEDT: track 83.3 -> 78.0 mm
- net /AUD_OUT_SUM: track 109.3 -> 111.9 mm
- net Net-(C63-Pad1): track 90.0 -> 92.4 mm
- net Net-(R49-Pad1): track 32.1 -> 31.0 mm
- net /SER_EECS: track 78.9 -> 79.6 mm
- net Net-(R51-Pad1): track 80.3 -> 80.9 mm

Commit message: daily
Parts:
- removed D10, D9: RB751V40T1G, Diode_SMD:D_SOD-323_HandSoldering
- removed R21: 100k, Resistor_SMD:R_0805_2012Metric_Pad1.20x1.40mm_HandSolder
- removed R64, R71, R72, R77: 10k, Resistor_SMD:R_0805_2012Metric_Pad1.20x1.40mm_HandSolder
- removed TP12: OPAMP_BIAS, TestPoint:TestPoint_Pad_D2.0mm
- removed U23: LMV321IDBVR, Package_TO_SOT_SMD:SOT-23-5_HandSoldering
- added SW8: SW_SPDT, switches_spdt_dpdt:Ninigi_MSS-2235S, F.Cu at (129.9, 101.9)
- added U16: 74AHCT1G04, Package_TO_SOT_SMD:SOT-23-5_HandSoldering, F.Cu at (181.3, 88.8)
- SW4, SW5: value SW_DIP_x04 -> A6H-4101
- U14: value 93CxxC -> AT93C46D
- moved R25 56.6 mm to (187.6, 99.8)
- moved C61 8.42 mm to (115.7, 65.7)
- moved Q5 7.90 mm to (123.8, 94.2), turned to -90 degrees
- moved C46 6.46 mm to (112.2, 63.2), turned to 180 degrees
- moved R80 6.39 mm to (118.8, 83.0), turned to 180 degrees
- moved SW6 5.46 mm to (127.4, 87.4)
- moved C60 5.20 mm to (120.8, 67.3), turned to 0 degrees
- moved U18 5.00 mm to (123.2, 76.5), turned to 90 degrees
- moved R66 4.31 mm to (118.3, 78.9)
- moved R60 4.10 mm to (117.9, 63.2)
- moved C62 3.29 mm to (123.2, 69.6), turned to 0 degrees
- moved R79 2.85 mm to (126.2, 99.6), turned to 0 degrees
- moved TP8 1.93 mm to (135.3, 76.0)
- moved R68 1.48 mm to (112.0, 66.2), turned to -90 degrees
- moved R63 0.15 mm to (134.1, 73.4), turned to -90 degrees
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Connections:
- C41 pad 1: /SER_VCCIO -> VCC
- C47 pad 1: /SER_VCCIO -> VCC
- C53 pad 1: /SER_VCCIO -> VCC
- C56 pad 1: /SER_VCCIO -> VCC
- L6 pad 2: /SER_VCCIO -> VCC
- Q4 pad 1: Net-(Q4-Pad1) -> /PTT_CTRL_SW
- R25 pad 2: /SER_VCCIO -> VCC
- R27 pad 1: /SER_VCCIO -> VCC
- R28 pad 1: /SER_VCCIO -> VCC
- R29 pad 2: /SER_VCCIO -> VCC
- R49 pad 2: /SER_VCCIO -> VCC
- R51 pad 2: /SER_VCCIO -> VCC
- R52 pad 2: /SER_VCCIO -> VCC
- R63 pad 1: /PTT_CTRL -> /PTT_CTRL_SW
- R63 pad 2: Net-(Q4-Pad1) -> Net-(R63-Pad2)
- R65 pad 2: /SER_VCCIO -> VCC
- R66 pad 2: /SER_VCCIO -> VCC
- R67 pad 2: Net-(R67-Pad2) -> Net-(C62-Pad1)
- R68 pad 2: Net-(R67-Pad2) -> Net-(C62-Pad1)
- SW3 pad 1: unconnected-(SW3-Pad1) -> /~{PTT_CTRL}
- SW3 pad 2: /PTT_CTRL -> Net-(R63-Pad2)
- SW3 pad 3: /SER_VCCIO -> /PTT_CTRL
- U11 pad 8: /SER_VCCIO -> VCC
- U14 pad 6: /SER_VCCIO -> VCC
- U14 pad 8: /SER_VCCIO -> VCC
- U17 pad 20: /SER_VCCIO -> VCC
- U17 pad 31: /SER_VCCIO -> VCC
- U17 pad 42: /SER_VCCIO -> VCC
- U17 pad 50: /SER_VCCIO -> VCC
- U17 pad 56: /SER_VCCIO -> VCC
- U18 pad 4: /SER_VCCIO -> VCC
Routing:
- net /SER_VCCIO: track 280.7 -> 0.00 mm, vias 10 -> 0
- net VCC: track 0.00 -> 266.7 mm, vias 0 -> 12
- net /PTT_CTRL: track 116.7 -> 95.9 mm, vias 5 -> 6
- net Net-(R71-Pad1): track 18.6 -> 0.00 mm, vias 2 -> 0
- net Net-(R63-Pad2): track 0.00 -> 18.5 mm, vias 0 -> 1
- net /AUD_VBUS: track 44.3 -> 29.7 mm, vias 2 -> 1
- net Net-(R64-Pad1): track 13.3 -> 0.00 mm, vias 2 -> 0
- net Net-(Q5-Pad2): track 2.90 -> 14.4 mm, vias 0 -> 2
- net /SER_B_RXD_IN: track 116.6 -> 105.4 mm, vias 3 -> 5
- net Net-(C61-Pad1): track 13.5 -> 2.41 mm, vias 2 -> 0
- net Net-(R79-Pad1): track 8.28 -> 0.00 mm
- net Net-(Q4-Pad3): track 42.9 -> 36.0 mm, vias 5 -> 4
- net Net-(Q5-Pad3): track 4.17 -> 11.0 mm
- net Net-(R67-Pad2): track 6.43 -> 0.00 mm
- net Net-(SW6-Pad2): track 13.3 -> 7.50 mm, vias 1 -> 0
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Other:
- board text added: "USB to Land Mobile Radio interface Revision B"
- board text removed: "USB to Land Mobile Radio interface Revision A"

Commit message: hw revision b done
Parts:
- removed R25: 2k2, Resistor_SMD:R_0805_2012Metric_Pad1.20x1.40mm_HandSolder
- moved U16 48.4 mm to (134.3, 100.5)
- moved R29 12.5 mm to (129.7, 89.3)
- moved R39 0.29 mm to (143.7, 102.0)
- moved R35 0.28 mm to (146.2, 103.8)
- moved C23 0.14 mm to (146.7, 100.5)
Connections:
- net Net-(R25-Pad1) renamed /SER_B_RXD_RS
- R29 pad 1: Net-(R29-Pad1) -> /SER_B_RXD_IN
- SW8 pad 1: Net-(R29-Pad1) -> /SER_B_RXD_TTL
- U11 pad 7: Net-(R29-Pad1) -> /SER_B_RXD_TTL
Routing:
- net GND: track 1091.6 -> 1155.3 mm, vias 127 -> 134
- net /~{PTT_CTRL}: track 0.00 -> 39.4 mm, vias 0 -> 3
- net /AF_FRM_RADIO_PREINS: track 90.4 -> 123.2 mm, vias 4 -> 5
- net Net-(R63-Pad2): track 18.5 -> 46.9 mm, vias 1 -> 3
- net /AUD_IN_SUM: track 92.8 -> 118.0 mm
- net VCC: track 266.7 -> 250.9 mm
- net Net-(R79-Pad1): track 0.00 -> 15.6 mm, vias 0 -> 1
- net Net-(R79-Pad2): track 0.00 -> 13.0 mm
- net /SER_EEDT: track 78.0 -> 89.9 mm, vias 2 -> 3
- net /PTT_CTRL: track 95.9 -> 104.9 mm
- net Net-(R29-Pad1): track 8.60 -> 0.00 mm
- net /SER_B_RXD_TTL: track 0.00 -> 5.72 mm
- net Net-(D12-Pad2): track 19.5 -> 14.0 mm
- net /SER_B_RXD_IN: track 105.4 -> 110.0 mm
- net Net-(SW6-Pad2): track 7.50 -> 12.1 mm
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Other:
- board text added: "RS232"
- board text added: "TTL"
